Commit message: changing urdfs to point to meshes in stl instead of dae

File: baxter_description/urdf/baxter_base/baxter_base.urdf.xacro (robot description, xacro)
@@ -12,5 +12,5 @@
       <origin rpy="0 0 0" xyz="0 0 0"/>
       <geometry>
-        <mesh filename="package://baxter_description/meshes/torso/base_link.DAE"/>
+        <mesh filename="package://baxter_description/meshes/torso/base_link.STL"/>
       </geometry>
       <material name="darkgray">
@@ -21,5 +21,5 @@
       <origin rpy="0 0 0" xyz="0 0 0"/>
       <geometry>
-        <mesh filename="package://baxter_description/meshes/torso/base_link_collision.DAE"/>
+        <mesh filename="package://baxter_description/meshes/torso/base_link_collision.STL"/>
       </geometry>
     </collision>
@@ -48,5 +48,5 @@
       <origin rpy="0 0 0" xyz="0 0 .00953"/>
       <geometry>
-        <mesh filename="package://baxter_description/meshes/head/H0.DAE"/>
+        <mesh filename="package://baxter_description/meshes/head/H0.STL"/>
       </geometry>
       <material name="darkgray">
@@ -92,5 +92,5 @@
       <origin rpy="0 -1.57079632679 0" xyz="0 -.00953 -.0347"/>
       <geometry>
-        <mesh filename="package://baxter_description/meshes/head/H1.DAE"/>
+        <mesh filename="package://baxter_description/meshes/head/H1.STL"/>
       </geometry>
       <material name="darkred">
@@ -256,5 +256,5 @@
       <origin rpy="0 0 0" xyz="0 0 0"/>
       <geometry>
-        <mesh filename="package://baxter_description/meshes/upper_shoulder/S0.DAE"/>
+        <mesh filename="package://baxter_description/meshes/upper_shoulder/S0.STL"/>
       </geometry>
       <material name="darkred">
@@ -278,5 +278,5 @@
       <origin rpy="0 0 0" xyz="0 0 0"/>
       <geometry>
-        <mesh filename="package://baxter_description/meshes/lower_shoulder/S1.DAE"/>
+        <mesh filename="package://baxter_description/meshes/lower_shoulder/S1.STL"/>
       </geometry>
       <material name="darkred">
@@ -300,5 +300,5 @@
       <origin rpy="0 0 0" xyz="0 0 0"/>
       <geometry>
-        <mesh filename="package://baxter_description/meshes/upper_elbow/E0.DAE"/>
+        <mesh filename="package://baxter_description/meshes/upper_elbow/E0.STL"/>
       </geometry>
       <material name="darkred">
@@ -335,5 +335,5 @@
       <origin rpy="0 0 0" xyz="0 0 0"/>
       <geometry>
-        <mesh filename="package://baxter_description/meshes/lower_elbow/E1.DAE"/>
+        <mesh filename="package://baxter_description/meshes/lower_elbow/E1.STL"/>
       </geometry>
       <material name="darkred">
@@ -357,5 +357,5 @@
       <origin rpy="0 0 0" xyz="0 0 0"/>
       <geometry>
-        <mesh filename="package://baxter_description/meshes/upper_forearm/W0.DAE"/>
+        <mesh filename="package://baxter_description/meshes/upper_forearm/W0.STL"/>
       </geometry>
       <material name="darkred">
@@ -399,5 +399,5 @@
       <origin rpy="0 0 0" xyz="0 0 0"/>
       <geometry>
-        <mesh filename="package://baxter_description/meshes/lower_forearm/W1.DAE"/>
+        <mesh filename="package://baxter_description/meshes/lower_forearm/W1.STL"/>
       </geometry>
       <material name="darkred">
@@ -421,5 +421,5 @@
       <origin rpy="0 0 0" xyz="0 0 0"/>
       <geometry>
-        <mesh filename="package://baxter_description/meshes/wrist/W2.DAE"/>
+        <mesh filename="package://baxter_description/meshes/wrist/W2.STL"/>
       </geometry>
       <material name="lightgrey">
@@ -624,5 +624,5 @@
       <origin rpy="0 0 0" xyz="0 0 0"/>
       <geometry>
-        <mesh filename="package://baxter_description/meshes/upper_shoulder/S0.DAE"/>
+        <mesh filename="package://baxter_description/meshes/upper_shoulder/S0.STL"/>
       </geometry>
       <material name="darkred">
@@ -646,5 +646,5 @@
       <origin rpy="0 0 0" xyz="0 0 0"/>
       <geometry>
-        <mesh filename="package://baxter_description/meshes/lower_shoulder/S1.DAE"/>
+        <mesh filename="package://baxter_description/meshes/lower_shoulder/S1.STL"/>
       </geometry>
       <material name="darkred">
@@ -668,5 +668,5 @@
       <origin rpy="0 0 0" xyz="0 0 0"/>
       <geometry>
-        <mesh filename="package://baxter_description/meshes/upper_elbow/E0.DAE"/>
+        <mesh filename="package://baxter_description/meshes/upper_elbow/E0.STL"/>
       </geometry>
       <material name="darkred">
@@ -703,5 +703,5 @@
       <origin rpy="0 0 0" xyz="0 0 0"/>
       <geometry>
-        <mesh filename="package://baxter_description/meshes/lower_elbow/E1.DAE"/>
+        <mesh filename="package://baxter_description/meshes/lower_elbow/E1.STL"/>
       </geometry>
       <material name="darkred">
@@ -725,5 +725,5 @@
       <origin rpy="0 0 0" xyz="0 0 0"/>
       <geometry>
-        <mesh filename="package://baxter_description/meshes/upper_forearm/W0.DAE"/>
+        <mesh filename="package://baxter_description/meshes/upper_forearm/W0.STL"/>
       </geometry>
       <material name="darkred">
@@ -767,5 +767,5 @@
       <origin rpy="0 0 0" xyz="0 0 0"/>
       <geometry>
-        <mesh filename="package://baxter_description/meshes/lower_forearm/W1.DAE"/>
+        <mesh filename="package://baxter_description/meshes/lower_forearm/W1.STL"/>
       </geometry>
       <material name="darkred">
@@ -789,5 +789,5 @@
       <origin rpy="0 0 0" xyz="0 0 0"/>
       <geometry>
-        <mesh filename="package://baxter_description/meshes/wrist/W2.DAE"/>
+        <mesh filename="package://baxter_description/meshes/wrist/W2.STL"/>
       </geometry>
       <material name="lightgrey">

File: baxter_description/urdf/pedestal/pedestal.xacro (robot description, xacro)
@@ -7,5 +7,5 @@
       <origin rpy="0 0 0" xyz="0 0 0"/>
       <geometry>
-        <mesh filename="package://baxter_description/meshes/base/PEDESTAL.DAE"/>
+        <mesh filename="package://baxter_description/meshes/base/PEDESTAL.STL"/>
       </geometry>
       <material name="darkgray">
@@ -16,5 +16,5 @@
       <origin rpy="0 0 0" xyz="0 0 0"/>
       <geometry>
-        <mesh filename="package://baxter_description/meshes/base/pedestal_link_collision.DAE"/>
+        <mesh filename="package://baxter_description/meshes/base/pedestal_link_collision.STL"/>
       </geometry>
     </collision>

File: rethink_ee_description/urdf/electric_gripper/fingers/basic_hard_tip.xacro (robot description, xacro)
@@ -10,5 +10,5 @@
         <origin rpy="0 0 ${pi*(g_reflect+1)/2}" xyz="0 0 0"/>
         <geometry>
-          <mesh filename="package://rethink_ee_description/meshes/electric_gripper/fingers/basic_hard_tip.DAE" />
+          <mesh filename="package://rethink_ee_description/meshes/electric_gripper/fingers/basic_hard_tip.STL" />
         </geometry>
       </visual>

File: rethink_ee_description/urdf/electric_gripper/fingers/basic_soft_tip.xacro (robot description, xacro)
@@ -10,5 +10,5 @@
         <origin rpy="0 0 ${pi*(g_reflect+1)/2}" xyz="0 0 0"/>
         <geometry>
-          <mesh filename="package://rethink_ee_description/meshes/electric_gripper/fingers/basic_soft_tip.DAE" />
+          <mesh filename="package://rethink_ee_description/meshes/electric_gripper/fingers/basic_soft_tip.STL" />
         </geometry>
       </visual>

File: rethink_ee_description/urdf/electric_gripper/fingers/extended_narrow.xacro (robot description, xacro)
@@ -8,5 +8,5 @@
         <origin rpy="0 0 ${-pi/2*(reflect+1)}" xyz="0 0 0"/>
         <geometry>
-          <mesh filename="package://rethink_ee_description/meshes/electric_gripper/fingers/extended_narrow.DAE" />
+          <mesh filename="package://rethink_ee_description/meshes/electric_gripper/fingers/extended_narrow.STL" />
         </geometry>
       </visual>

File: rethink_ee_description/urdf/electric_gripper/fingers/extended_wide.xacro (robot description, xacro)
@@ -8,5 +8,5 @@
         <origin rpy="0 0 ${-pi/2*(reflect+1)}" xyz="0 0 0"/>
         <geometry>
-          <mesh filename="package://rethink_ee_description/meshes/electric_gripper/fingers/extended_wide.DAE" />
+          <mesh filename="package://rethink_ee_description/meshes/electric_gripper/fingers/extended_wide.STL" />
         </geometry>
       </visual>

File: rethink_ee_description/urdf/electric_gripper/fingers/half_round_tip.xacro (robot description, xacro)
@@ -10,5 +10,5 @@
         <origin rpy="0 0 ${pi*(g_reflect+1)/2}" xyz="0 0 0"/>
         <geometry>
-          <mesh filename="package://rethink_ee_description/meshes/electric_gripper/fingers/half_round_tip.DAE" />
+          <mesh filename="package://rethink_ee_description/meshes/electric_gripper/fingers/half_round_tip.STL" />
         </geometry>
       </visual>

File: rethink_ee_description/urdf/electric_gripper/fingers/paddle_tip.xacro (robot description, xacro)
@@ -10,5 +10,5 @@
         <origin rpy="0 0 ${pi*(g_reflect+1)/2}" xyz="0 0 0"/>
         <geometry>
-          <mesh filename="package://rethink_ee_description/meshes/electric_gripper/fingers/paddle_tip.DAE" />
+          <mesh filename="package://rethink_ee_description/meshes/electric_gripper/fingers/paddle_tip.STL" />
         </geometry>
       </visual>

File: rethink_ee_description/urdf/electric_gripper/fingers/standard_narrow.xacro (robot description, xacro)
@@ -8,5 +8,5 @@
         <origin rpy="0 0 ${-pi/2*(reflect+1)}" xyz="0 0 0"/>
         <geometry>
-          <mesh filename="package://rethink_ee_description/meshes/electric_gripper/fingers/standard_narrow.DAE" />
+          <mesh filename="package://rethink_ee_description/meshes/electric_gripper/fingers/standard_narrow.STL" />
         </geometry>
       </visual>

File: rethink_ee_description/urdf/electric_gripper/fingers/standard_wide.xacro (robot description, xacro)
@@ -8,5 +8,5 @@
         <origin rpy="0 0 ${-pi/2*(reflect+1)}" xyz="0 0 0"/>
         <geometry>
-          <mesh filename="package://rethink_ee_description/meshes/electric_gripper/fingers/standard_wide.DAE" />
+          <mesh filename="package://rethink_ee_description/meshes/electric_gripper/fingers/standard_wide.STL" />
         </geometry>
       </visual>

File: rethink_ee_description/urdf/electric_gripper/rethink_electric_gripper.xacro (robot description, xacro)
@@ -8,5 +8,5 @@
         <origin rpy="${-pi/2} ${pi} 0" xyz="0 0 0"/>
         <geometry>
-          <mesh filename="package://rethink_ee_description/meshes/electric_gripper/electric_gripper_base.DAE"/>
+          <mesh filename="package://rethink_ee_description/meshes/electric_gripper/electric_gripper_base.STL"/>
         </geometry>
       </visual>
